Commit message: Rename packages

File: leo2_description/urdf/leo2_sim.urdf.xacro (robot description, xacro)
@@ -1,9 +1,9 @@
 <?xml version="1.0"?>
 <robot xmlns:xacro="http://ros.org/wiki/xacro"
-       name="leo_sim">
+       name="leo2_sim">
   <xacro:arg name="fixed" default="false"/>
   <xacro:arg name="robot_ns" default=""/>
-  <xacro:include filename="$(find leo_description)/urdf/macros.xacro"/>
-  <xacro:leo_sim robot_ns="$(arg robot_ns)"
+  <xacro:include filename="$(find leo2_description)/urdf/macros.xacro"/>
+  <xacro:leo2_sim robot_ns="$(arg robot_ns)"
                  fixed="$(arg fixed)"/>
 </robot>

File: leo2_description/urdf/macros.xacro (robot description, xacro)
@@ -1,5 +1,5 @@
 <?xml version="1.0" encoding="utf-8"?>
 <robot xmlns:xacro="http://www.ros.org/wiki/xacro">
-  <xacro:macro name="leo"
+  <xacro:macro name="leo2"
                params="default_antenna:=true
                        rockers_fixed:=true
@@ -20,10 +20,10 @@
         <visual>
           <geometry>
-            <mesh filename="package://leo_description/models/Rocker.dae"/>
+            <mesh filename="package://leo2_description/models/Rocker.dae"/>
           </geometry>
         </visual>
         <collision>
           <geometry>
-            <mesh filename="package://leo_description/models/Rocker_outline.stl"/>
+            <mesh filename="package://leo2_description/models/Rocker_outline.stl"/>
           </geometry>
         </collision>
@@ -42,5 +42,5 @@
         <visual>
           <geometry>
-            <mesh filename="package://leo_description/models/Wheel${model}.dae"/>
+            <mesh filename="package://leo2_description/models/Wheel${model}.dae"/>
           </geometry>
         </visual>
@@ -59,5 +59,5 @@
         <collision>
           <geometry>
-            <mesh filename="package://leo_description/models/Wheel_outline.stl"/>
+            <mesh filename="package://leo2_description/models/Wheel_outline.stl"/>
           </geometry>
         </collision>
@@ -79,10 +79,10 @@
       <visual>
         <geometry>
-          <mesh filename="package://leo_description/models/Chassis.dae"/>
+          <mesh filename="package://leo2_description/models/Chassis.dae"/>
         </geometry>
       </visual>
       <collision>
         <geometry>
-          <mesh filename="package://leo_description/models/Chassis_outline.stl"/>
+          <mesh filename="package://leo2_description/models/Chassis_outline.stl"/>
         </geometry>
       </collision>
@@ -106,5 +106,5 @@
         <visual>
           <geometry>
-            <mesh filename="package://leo_description/models/Antenna.dae"/>
+            <mesh filename="package://leo2_description/models/Antenna.dae"/>
           </geometry>
         </visual>
@@ -207,5 +207,5 @@
   </xacro:macro>
   <!-- LEO GAZEBO -->
-  <xacro:macro name="leo_gazebo"
+  <xacro:macro name="leo2_gazebo"
                params="robot_ns:=''">
     <xacro:property name="link_prefix" value=""/>
@@ -385,9 +385,9 @@
         <robot_param>robot_description</robot_param>
         <robot_param_node>robot_state_publisher</robot_param_node>
-        <parameters>package://leo_description/config/controllers.yaml</parameters>
+        <parameters>package://leo2_description/config/controllers.yaml</parameters>
       </plugin>
     </gazebo>
   </xacro:macro>
-  <xacro:macro name="leo_sim"
+  <xacro:macro name="leo2_sim"
                params="default_antenna:=true
                        fixed:=false
@@ -397,8 +397,8 @@
       <xacro:property name="link_prefix" value="${robot_ns}/"/>
     </xacro:if>
-    <xacro:leo default_antenna="${default_antenna}"
+    <xacro:leo2 default_antenna="${default_antenna}"
                rockers_fixed="false"
                link_prefix="${link_prefix}"/>
-    <xacro:leo_gazebo robot_ns="${robot_ns}"/>
+    <xacro:leo2_gazebo robot_ns="${robot_ns}"/>
     <xacro:if value="${fixed}">
       <link name="world"/>
