Commit message: Add zed2 to description

File: leo2_description/urdf/macros.xacro (robot description, xacro)
@@ -1,4 +1,5 @@
 <?xml version="1.0" encoding="utf-8"?>
 <robot xmlns:xacro="http://www.ros.org/wiki/xacro">
+  <xacro:include filename="$(find leo2_description)/urdf/include/zed_macro.xacro"/>
   <xacro:macro name="leo2"
                params="default_antenna:=true
@@ -8,4 +9,7 @@
                        joint_prefix:=''
                        imu_translation:='0.0628 -0.0314 -0.0393'">
+    <xacro:zed_camera name="${link_prefix}zed2i" model="zed2i" parent="${link_prefix}base_link">
+      <origin xyz="0.151138 0.0 0.019725" rpy="0 0.0872664626 0" />
+    </xacro:zed_camera>
     <xacro:macro name="rocker_link" params="name">
       <link name="${link_prefix}rocker_${name}_link">

Commit message: Add oak camera description

File: leo2_description/urdf/macros.xacro (robot description, xacro)
@@ -1,5 +1,5 @@
 <?xml version="1.0" encoding="utf-8"?>
 <robot xmlns:xacro="http://www.ros.org/wiki/xacro">
-  <xacro:include filename="$(find leo2_description)/urdf/include/zed_macro.xacro"/>
+  <xacro:include filename="$(find leo2_description)/urdf/include/oak_macro.xacro"/>
   <xacro:macro name="leo2"
                params="default_antenna:=true
@@ -9,7 +9,7 @@
                        joint_prefix:=''
                        imu_translation:='0.0628 -0.0314 -0.0393'">
-    <xacro:zed_camera name="${link_prefix}zed2i" model="zed2i" parent="${link_prefix}base_link">
-      <origin xyz="0.151138 0.0 0.019725" rpy="0 0.0872664626 0" />
-    </xacro:zed_camera>
+    <xacro:oak_camera parent="${link_prefix}base_link" base_frame="oak_base_link">
+      <origin xyz="0.1446 0.0 0.02476" rpy="0 0 0" />
+    </xacro:oak_camera>
     <xacro:macro name="rocker_link" params="name">
       <link name="${link_prefix}rocker_${name}_link">
