Commit message: Fix mesh paths

File: leo2_description/urdf/include/zed_macro.xacro (robot description, xacro)
@@ -66,5 +66,5 @@
         <origin xyz="${screw_offset_x} 0 0" rpy="0 0 0"/>
         <geometry>
-          <mesh filename="package://leo2_description/meshes/${model}.stl" />
+          <mesh filename="package://leo2_description/models/${model}.stl" />
         </geometry>
         <material name="${model}_mat" />
@@ -72,5 +72,5 @@
       <collision>
         <geometry>
-          <mesh filename="package://leo2_description/meshes/${model}.stl" />
+          <mesh filename="package://leo2_description/models/${model}.stl" />
         </geometry>
       </collision>
