Commit message: Remove capital letters from joint and link names

File: rapha_description/urdf/rapha_macros.xacro (robot description, xacro)
@@ -66,10 +66,10 @@
     </link>
     <link name="${link_prefix}mounting_plate_frame"/>
-    <xacro:servo_link name="L"/>
-    <xacro:servo_link name="R"/>
-    <xacro:wheel_link name="FL"/>
-    <xacro:wheel_link name="RL"/>
-    <xacro:wheel_link name="FR"/>
-    <xacro:wheel_link name="RR"/>
+    <xacro:servo_link name="l"/>
+    <xacro:servo_link name="r"/>
+    <xacro:wheel_link name="fl"/>
+    <xacro:wheel_link name="rl"/>
+    <xacro:wheel_link name="fr"/>
+    <xacro:wheel_link name="rr"/>
     <link name="${link_prefix}imu_frame"/>
     <!-- JOINTS -->
@@ -81,46 +81,46 @@
       </joint>
     </xacro:if>
-    <joint name="${joint_prefix}servo_L_joint" type="revolute">
+    <joint name="${joint_prefix}servo_l_joint" type="revolute">
       <origin xyz="-0.37943 0.1899 -0.022433" rpy="0 0 0"/>
       <parent link="${link_prefix}base_link"/>
-      <child link="${link_prefix}servo_L_link"/>
+      <child link="${link_prefix}servo_l_link"/>
       <axis xyz="0 0 -1"/>
       <limit effort="100.0" lower="-1.5708" upper="1.5708" velocity="100.0"/>
     </joint>
-    <joint name="${joint_prefix}servo_R_joint" type="revolute">
+    <joint name="${joint_prefix}servo_r_joint" type="revolute">
       <origin xyz="-0.37943 -0.1899 -0.022433" rpy="0 0 ${pi}"/>
       <parent link="${link_prefix}base_link"/>
-      <child link="${link_prefix}servo_R_link"/>
+      <child link="${link_prefix}servo_r_link"/>
       <axis xyz="0 0 -1"/>
       <limit effort="100.0" lower="-1.5708" upper="1.5708" velocity="100.0"/>
     </joint>
-    <joint name="${joint_prefix}wheel_FL_joint" type="continuous">
+    <joint name="${joint_prefix}wheel_fl_joint" type="continuous">
       <origin xyz="0 0.19402 -0.144756" rpy="0 0 0"/>
       <parent link="${link_prefix}base_link"/>
-      <child link="${link_prefix}wheel_FL_link"/>
+      <child link="${link_prefix}wheel_fl_link"/>
       <axis xyz="0 1 0"/>
       <limit effort="2.0" velocity="6.0"/>
       <dynamics friction="0.3125" damping="0.1"/>
     </joint>
-    <joint name="${joint_prefix}wheel_RL_joint" type="continuous">
+    <joint name="${joint_prefix}wheel_rl_joint" type="continuous">
       <origin xyz="0 0 -0.12392" rpy="0 0 0"/>
-      <parent link="${link_prefix}servo_L_link"/>
-      <child link="${link_prefix}wheel_RL_link"/>
+      <parent link="${link_prefix}servo_l_link"/>
+      <child link="${link_prefix}wheel_rl_link"/>
       <axis xyz="0 1 0"/>
       <limit effort="2.0" velocity="6.0"/>
       <dynamics friction="0.3125" damping="0.1"/>
     </joint>
-    <joint name="${joint_prefix}wheel_FR_joint" type="continuous">
+    <joint name="${joint_prefix}wheel_fr_joint" type="continuous">
       <origin xyz="0 -0.19402 -0.144756" rpy="0 0 ${pi}"/>
       <parent link="${link_prefix}base_link"/>
-      <child link="${link_prefix}wheel_FR_link"/>
+      <child link="${link_prefix}wheel_fr_link"/>
       <axis xyz="0 -1 0"/>
       <limit effort="2.0" velocity="6.0"/>
       <dynamics friction="0.3125" damping="0.1"/>
     </joint>
-    <joint name="${joint_prefix}wheel_RR_joint" type="continuous">
+    <joint name="${joint_prefix}wheel_rr_joint" type="continuous">
       <origin xyz="0 0 -0.12392" rpy="0 0 0"/>
-      <parent link="${link_prefix}servo_R_link"/>
-      <child link="${link_prefix}wheel_RR_link"/>
+      <parent link="${link_prefix}servo_r_link"/>
+      <child link="${link_prefix}wheel_rr_link"/>
       <axis xyz="0 -1 0"/>
       <limit effort="2.0" velocity="6.0"/>

Commit message: Add new URDF file for Rapha rover (#5)
* Add new URDF file for Rapha rover

* Improve collada materials visibility

* Remove capital letters from joint and link names

File: rapha_description/urdf/rapha_macros.xacro (robot description, xacro)
@@ -2,95 +2,45 @@
 <robot xmlns:xacro="http://www.ros.org/wiki/xacro">
   <xacro:include filename="$(find rapha_description)/urdf/include/oak_macro.xacro"/>
+  <xacro:include filename="$(find rapha_description)/urdf/include/laser_macro.xacro"/>
   <xacro:macro name="rapha"
-               params="default_antenna:=true
-                       rockers_fixed:=true
-                       footprint_link:=true
+               params="footprint_link:=true
                        link_prefix:=''
                        joint_prefix:=''
-                       imu_translation:='0.0628 -0.0314 -0.0393'
-                       mecanum_wheels:=false">
-    <xacro:oak_camera parent="${link_prefix}base_link" base_frame="${link_prefix}oak_base_link">
-      <origin xyz="0.1446 0.0 0.02476" rpy="0 0 0" />
+                       imu_translation:='-0.128 0 -0.0393'">
+    <!--TODO specify accurate imu translation-->
+    <xacro:oak_camera parent="${link_prefix}base_link" base_frame="${link_prefix}oak_base_frame">
+      <origin xyz="-0.05642 0.0 -0.076218" rpy="0 0 0" />
     </xacro:oak_camera>
-    <xacro:macro name="rocker_link" params="name">
-      <link name="${link_prefix}rocker_${name}_link">
-        <inertial>
-          <mass value="1.387336"/>
-          <origin xyz="0 0.01346 -0.06506"/>
-          <inertia
-            ixx="0.002956" ixy="-0.000001489324" ixz="-0.000008103407"
-            iyy="0.02924"  iyz="0.00007112"
-            izz="0.02832"/>
-        </inertial>
+    <xacro:rplidar_s3 parent="${link_prefix}base_link">
+      <origin xyz="-0.062106 0.0 0.011588" />
+    </xacro:rplidar_s3>
+    <xacro:macro name="servo_link" params="name">
+      <link name="${link_prefix}servo_${name}_link">
         <visual>
+          <origin xyz="0 0 0" rpy="0 0 ${pi/2}"/>
           <geometry>
-            <mesh filename="package://rapha_description/models/Rocker.dae"/>
+            <mesh filename="package://rapha_description/models/servo.dae"/>
           </geometry>
         </visual>
         <collision>
+          <origin xyz="0 0 0" rpy="0 0 0"/>
           <geometry>
-            <mesh filename="package://rapha_description/models/Rocker_outline.stl"/>
+            <mesh filename="package://rapha_description/models/servo_outline.stl"/>
           </geometry>
         </collision>
       </link>
     </xacro:macro>
-    <xacro:macro name="wheel_link" params="name model">
+    <xacro:macro name="wheel_link" params="name">
       <link name="${link_prefix}wheel_${name}_link">
-        <inertial>
-          <mass value="0.283642"/>
-          <origin xyz="0 0.030026 0"/>
-          <inertia
-            ixx="0.000391"  ixy="0.00000123962" ixz="5.52582e-7"
-            iyy="0.0004716" iyz="-0.000002082042"
-            izz="0.000391"/>
-        </inertial>
         <visual>
+          <origin xyz="0 0 0" rpy="0 0 ${pi/2}"/>
           <geometry>
-            <mesh filename="package://rapha_description/models/Wheel${model}.dae"/>
+            <mesh filename="package://rapha_description/models/wheel.dae"/>
           </geometry>
         </visual>
         <collision>
-          <origin xyz="0 0.04485 0" rpy="${pi/2} 0 0"/>
+          <origin xyz="0 0 0" rpy="${pi/2} 0 0"/>
           <geometry>
-            <cylinder radius="0.057" length="0.07"/>
-          </geometry>
-        </collision>
-        <collision>
-          <origin xyz="0 0.04485 0" rpy="${pi/2} 0 0"/>
-          <geometry>
-            <cylinder radius="0.0625" length="0.04"/>
-          </geometry>
-        </collision>
-        <collision>
-          <geometry>
-            <mesh filename="package://rapha_description/models/Wheel_outline.stl"/>
-          </geometry>
-        </collision>
-      </link>
-    </xacro:macro>
-    <xacro:macro name="mecanum_wheel_link" params="name model">
-      <link name="${link_prefix}wheel_${name}_link">
-        <inertial>
-          <mass value="0.672214"/>
-          <origin xyz="0 -0.036852 0"/>
-          <inertia
-            ixx="0.0009778"  ixy="-8.10228e-7" ixz="3.2e-11"
-            iyy="0.001321" iyz="5.7e-11"
-            izz="0.0009773"/>
-        </inertial>
-        <visual>
-          <geometry>
-            <mesh filename="package://rapha_description/models/WheelMecanum${model}.dae"/>
-          </geometry>
-        </visual>
-        <collision>
-          <origin xyz="0 -0.0317 0" rpy="${pi/2} 0 0"/>
-          <geometry>
-            <cylinder radius="0.0635" length="0.0515"/>
-          </geometry>
-        </collision>
-        <collision>
-          <geometry>
-            <mesh filename="package://rapha_description/models/Mecanum_wheel_outline.stl"/>
+            <cylinder radius="0.091" length="0.088"/>
           </geometry>
         </collision>
@@ -102,162 +52,78 @@
     </xacro:if>
     <link name="${link_prefix}base_link">
-      <inertial>
-        <mass value="1.584994"/>
-        <origin xyz="-0.019662 0.011643 -0.031802"/>
-        <inertia
-          ixx="0.01042" ixy="0.001177" ixz="-0.0008871"
-          iyy="0.01045" iyz="0.0002226"
-          izz="0.01817"/>
-      </inertial>
       <visual>
+        <origin xyz="-0.074211 0 -0.031076" rpy="0 0 ${pi/2}"/>
         <geometry>
-          <mesh filename="package://rapha_description/models/Chassis.dae"/>
+          <mesh filename="package://rapha_description/models/rapha_base_link.dae"/>
         </geometry>
       </visual>
       <collision>
+        <origin xyz="0 0 -0.031076" rpy="0 0 0"/>
         <geometry>
-          <mesh filename="package://rapha_description/models/Chassis_outline.stl"/>
+          <mesh filename="package://rapha_description/models/rapha_outline.stl"/>
         </geometry>
       </collision>
     </link>
-    <xacro:rocker_link name="L"/>
-    <xacro:rocker_link name="R"/>
-    <xacro:if value="${mecanum_wheels}">
-      <xacro:mecanum_wheel_link name="FL" model="B"/>
-      <xacro:mecanum_wheel_link name="RL" model="A"/>
-      <xacro:mecanum_wheel_link name="FR" model="A"/>
-      <xacro:mecanum_wheel_link name="RR" model="B"/>
-    </xacro:if>
-    <xacro:unless value="${mecanum_wheels}">
-      <xacro:wheel_link name="FL" model="A"/>
-      <xacro:wheel_link name="RL" model="A"/>
-      <xacro:wheel_link name="FR" model="B"/>
-      <xacro:wheel_link name="RR" model="B"/>
-    </xacro:unless>
-    <xacro:if value="${default_antenna}">
-      <link name="${link_prefix}antenna_link">
-        <inertial>
-          <mass value="0.001237"/>
-          <origin xyz="0 0 0.028828"/>
-          <inertia
-            ixx="2.5529e-7" ixy="0.0" ixz="0.0"
-            iyy="2.5529e-7" iyz="0.0"
-            izz="1.354e-8"/>
-        </inertial>
-        <visual>
-          <geometry>
-            <mesh filename="package://rapha_description/models/Antenna.dae"/>
-          </geometry>
-        </visual>
-        <collision>
-          <origin xyz="0 0 0.028"/>
-          <geometry>
-            <cylinder radius="0.0055" length="0.056"/>
-          </geometry>
-        </collision>
-      </link>
-    </xacro:if>
-    <link name="${link_prefix}camera_frame"/>
-    <link name="${link_prefix}camera_optical_frame"/>
+    <link name="${link_prefix}mounting_plate_frame"/>
+    <xacro:servo_link name="l"/>
+    <xacro:servo_link name="r"/>
+    <xacro:wheel_link name="fl"/>
+    <xacro:wheel_link name="rl"/>
+    <xacro:wheel_link name="fr"/>
+    <xacro:wheel_link name="rr"/>
     <link name="${link_prefix}imu_frame"/>
     <!-- JOINTS -->
     <xacro:if value="${footprint_link}">
       <joint name="${joint_prefix}base_joint" type="fixed">
-        <origin xyz="0 0 0.19783" rpy="0 0 0"/>
+        <origin xyz="0 0 0.235756" rpy="0 0 0"/>
         <parent link="${link_prefix}base_footprint"/>
         <child link="${link_prefix}base_link"/>
       </joint>
     </xacro:if>
-    <xacro:if value="${rockers_fixed}">
-      <xacro:property name="rockers_joint_type" value="fixed"/>
-    </xacro:if>
-    <xacro:unless value="${rockers_fixed}">
-      <xacro:property name="rockers_joint_type" value="revolute"/>
-    </xacro:unless>
-    <joint name="${joint_prefix}rocker_L_joint" type="${rockers_joint_type}">
-      <origin xyz="0.00263 0.14167 -0.04731" rpy="0 0 ${pi}"/>
+    <joint name="${joint_prefix}servo_l_joint" type="revolute">
+      <origin xyz="-0.37943 0.1899 -0.022433" rpy="0 0 0"/>
       <parent link="${link_prefix}base_link"/>
-      <child link="${link_prefix}rocker_L_link"/>
+      <child link="${link_prefix}servo_l_link"/>
+      <axis xyz="0 0 -1"/>
+      <limit effort="100.0" lower="-1.5708" upper="1.5708" velocity="100.0"/>
+    </joint>
+    <joint name="${joint_prefix}servo_r_joint" type="revolute">
+      <origin xyz="-0.37943 -0.1899 -0.022433" rpy="0 0 ${pi}"/>
+      <parent link="${link_prefix}base_link"/>
+      <child link="${link_prefix}servo_r_link"/>
+      <axis xyz="0 0 -1"/>
+      <limit effort="100.0" lower="-1.5708" upper="1.5708" velocity="100.0"/>
+    </joint>
+    <joint name="${joint_prefix}wheel_fl_joint" type="continuous">
+      <origin xyz="0 0.19402 -0.144756" rpy="0 0 0"/>
+      <parent link="${link_prefix}base_link"/>
+      <child link="${link_prefix}wheel_fl_link"/>
       <axis xyz="0 1 0"/>
-      <limit effort="100.0" lower="-0.24" upper="0.24" velocity="100.0"/>
-      <dynamics friction="1.0" damping="0.1"/>
+      <limit effort="2.0" velocity="6.0"/>
+      <dynamics friction="0.3125" damping="0.1"/>
     </joint>
-    <joint name="${joint_prefix}rocker_R_joint" type="${rockers_joint_type}">
-      <origin xyz="0.00263 -0.14167 -0.04731" rpy="0 0 0"/>
+    <joint name="${joint_prefix}wheel_rl_joint" type="continuous">
+      <origin xyz="0 0 -0.12392" rpy="0 0 0"/>
+      <parent link="${link_prefix}servo_l_link"/>
+      <child link="${link_prefix}wheel_rl_link"/>
+      <axis xyz="0 1 0"/>
+      <limit effort="2.0" velocity="6.0"/>
+      <dynamics friction="0.3125" damping="0.1"/>
+    </joint>
+    <joint name="${joint_prefix}wheel_fr_joint" type="continuous">
+      <origin xyz="0 -0.19402 -0.144756" rpy="0 0 ${pi}"/>
       <parent link="${link_prefix}base_link"/>
-      <child link="${link_prefix}rocker_R_link"/>
-      <axis xyz="0 1 0"/>
-      <limit effort="100.0" lower="-0.24" upper="0.24" velocity="100.0"/>
-      <dynamics friction="1.0" damping="0.1"/>
-      <mimic joint="rocker_L_joint"/>
-    </joint>
-    <joint name="${joint_prefix}wheel_FL_joint" type="continuous">
-      <xacro:if value="${mecanum_wheels}">
-        <origin xyz="-0.15256 -0.00884 -0.08802" rpy="0 0 0"/>
-      </xacro:if>
-      <xacro:unless value="${mecanum_wheels}">
-        <origin xyz="-0.15256 -0.08214 -0.08802" rpy="0 0 0"/>
-      </xacro:unless>
-      <parent link="${link_prefix}rocker_L_link"/>
-      <child link="${link_prefix}wheel_FL_link"/>
+      <child link="${link_prefix}wheel_fr_link"/>
       <axis xyz="0 -1 0"/>
       <limit effort="2.0" velocity="6.0"/>
       <dynamics friction="0.3125" damping="0.1"/>
     </joint>
-    <joint name="${joint_prefix}wheel_RL_joint" type="continuous">
-      <xacro:if value="${mecanum_wheels}">
-        <origin xyz="0.15256 -0.00884 -0.08802" rpy="0 0 0"/>
-      </xacro:if>
-      <xacro:unless value="${mecanum_wheels}">
-        <origin xyz="0.15256 -0.08214 -0.08802" rpy="0 0 0"/>
-      </xacro:unless>
-      <parent link="${link_prefix}rocker_L_link"/>
-      <child link="${link_prefix}wheel_RL_link"/>
+    <joint name="${joint_prefix}wheel_rr_joint" type="continuous">
+      <origin xyz="0 0 -0.12392" rpy="0 0 0"/>
+      <parent link="${link_prefix}servo_r_link"/>
+      <child link="${link_prefix}wheel_rr_link"/>
       <axis xyz="0 -1 0"/>
       <limit effort="2.0" velocity="6.0"/>
       <dynamics friction="0.3125" damping="0.1"/>
-    </joint>
-    <joint name="${joint_prefix}wheel_FR_joint" type="continuous">
-      <xacro:if value="${mecanum_wheels}">
-        <origin xyz="0.15256 -0.00884 -0.08802" rpy="0 0 0"/>
-      </xacro:if>
-      <xacro:unless value="${mecanum_wheels}">
-        <origin xyz="0.15256 -0.08214 -0.08802" rpy="0 0 0"/>
-      </xacro:unless>
-      <parent link="${link_prefix}rocker_R_link"/>
-      <child link="${link_prefix}wheel_FR_link"/>
-      <axis xyz="0 1 0"/>
-      <limit effort="2.0" velocity="6.0"/>
-      <dynamics friction="0.3125" damping="0.1"/>
-    </joint>
-    <joint name="${joint_prefix}wheel_RR_joint" type="continuous">
-      <xacro:if value="${mecanum_wheels}">
-        <origin xyz="-0.15256 -0.00884 -0.08802" rpy="0 0 0"/>
-      </xacro:if>
-      <xacro:unless value="${mecanum_wheels}">
-        <origin xyz="-0.15256 -0.08214 -0.08802" rpy="0 0 0"/>
-      </xacro:unless>
-      <parent link="${link_prefix}rocker_R_link"/>
-      <child link="${link_prefix}wheel_RR_link"/>
-      <axis xyz="0 1 0"/>
-      <limit effort="2.0" velocity="6.0"/>
-      <dynamics friction="0.3125" damping="0.1"/>
-    </joint>
-    <xacro:if value="${default_antenna}">
-      <joint name="${joint_prefix}antenna_joint" type="fixed">
-        <origin xyz="-0.0052 0.056 -0.0065" rpy="0 0 0"/>
-        <parent link="${link_prefix}base_link"/>
-        <child link="${link_prefix}antenna_link"/>
-      </joint>
-    </xacro:if>
-    <joint name="${joint_prefix}camera_joint" type="fixed">
-      <origin xyz="0.0971 0 -0.0427" rpy="0 0.2094 0"/>
-      <parent link="${link_prefix}base_link"/>
-      <child link="${link_prefix}camera_frame"/>
-    </joint>
-    <joint name="${joint_prefix}camera_optical_joint" type="fixed">
-      <origin xyz="0 0 0" rpy="-${pi/2} 0.0 -${pi/2}"/>
-      <parent link="${link_prefix}camera_frame"/>
-      <child link="${link_prefix}camera_optical_frame"/>
     </joint>
     <joint name="${joint_prefix}imu_joint" type="fixed">
@@ -266,4 +132,9 @@
       <child link="${link_prefix}imu_frame"/>
     </joint>
+    <joint name="${joint_prefix}mounting_plate_joint" type="fixed">
+      <origin xyz="-0.216822 0 0" rpy="0 0 0"/>
+      <parent link="${link_prefix}base_link"/>
+      <child link="${link_prefix}mounting_plate_frame"/>
+    </joint>
   </xacro:macro>
 </robot>
