Commit message: Add sensor namespacing and odom publisher

File: raph_description/urdf/include/laser_macro.xacro (robot description, xacro)
@@ -2,10 +2,10 @@
 <robot name="sp3lidar" xmlns:xacro="http://ros.org/wiki/xacro">
   <xacro:macro name="rplidar_s3"
-    params="parent *origin">
-    <link name="laser_frame"/>
-    <joint name="laser_joint" type="fixed">
+    params="parent *origin namespace:=''">
+    <link name="${namespace}laser_frame"/>
+    <joint name="${namespace}laser_joint" type="fixed">
       <xacro:insert_block name="origin"/>
       <parent link="${parent}"/>
-      <child link="laser_frame"/>
+      <child link="${namespace}laser_frame"/>
     </joint>
   </xacro:macro>

File: raph_description/urdf/include/oak_macro.xacro (robot description, xacro)
@@ -2,58 +2,58 @@
 <robot name="depthai_camera" xmlns:xacro="http://ros.org/wiki/xacro">
   <xacro:macro name="oak_camera"
-    params="parent base_frame *origin r:=0.3 g:=0.3 b:=0.3 a:=0.8">
+    params="parent base_frame *origin r:=0.3 g:=0.3 b:=0.3 a:=0.8 namespace:=''">
     <xacro:property name="baseline" value="0.075" />
     <!-- base_link of the sensor-->
-    <link name="${base_frame}"/>
-    <joint name="oak_center_joint" type="fixed">
+    <link name="${namespace}${base_frame}"/>
+    <joint name="${namespace}oak_center_joint" type="fixed">
       <parent link="${parent}"/>
-      <child link="${base_frame}"/>
+      <child link="${namespace}${base_frame}"/>
       <xacro:insert_block name="origin" />
     </joint>
     <!-- IMU -->
-    <link name="oak_imu_frame" />
-    <joint name="oak_imu_joint" type="fixed">
-      <parent link="${base_frame}"/>
-      <child link="oak_imu_frame"/>
+    <link name="${namespace}oak_imu_frame" />
+    <joint name="${namespace}oak_imu_joint" type="fixed">
+      <parent link="${namespace}${base_frame}"/>
+      <child link="${namespace}oak_imu_frame"/>
       <origin xyz="0.0 -0.015 -0.013662" rpy="0.0 ${pi/2} 0.0" />
     </joint>
     <!-- RGB Camera -->
-    <link name="oak_rgb_camera_frame" />
-    <joint name="oak_rgb_camera_joint" type="fixed">
-      <parent link="${base_frame}"/>
-      <child link="oak_rgb_camera_frame"/>
+    <link name="${namespace}oak_rgb_camera_frame" />
+    <joint name="${namespace}oak_rgb_camera_joint" type="fixed">
+      <parent link="${namespace}${base_frame}"/>
+      <child link="${namespace}oak_rgb_camera_frame"/>
       <origin xyz="0 0 0" rpy="0 0 0" />
     </joint>
-    <link name="oak_rgb_camera_optical_frame"/>
-    <joint name="oak_rgb_camera_optical_joint" type="fixed">
+    <link name="${namespace}oak_rgb_camera_optical_frame"/>
+    <joint name="${namespace}oak_rgb_camera_optical_joint" type="fixed">
       <origin xyz="0 0 0" rpy="-${pi/2} 0.0 -${pi/2}"/>
-      <parent link="oak_rgb_camera_frame"/>
-      <child link="oak_rgb_camera_optical_frame"/>
+      <parent link="${namespace}oak_rgb_camera_frame"/>
+      <child link="${namespace}oak_rgb_camera_optical_frame"/>
     </joint>
     <!-- Left Camera -->
-    <link name="oak_left_camera_frame" />
-    <joint name="oak_left_camera_joint" type="fixed">
-      <parent link="${base_frame}"/>
-      <child link="oak_left_camera_frame"/>
+    <link name="${namespace}oak_left_camera_frame" />
+    <joint name="${namespace}oak_left_camera_joint" type="fixed">
+      <parent link="${namespace}${base_frame}"/>
+      <child link="${namespace}oak_left_camera_frame"/>
       <origin xyz="0 ${baseline/2} 0" rpy="0 0 0" />
     </joint>
-    <link name="oak_left_camera_optical_frame"/>
-    <joint name="oak_left_camera_optical_joint" type="fixed">
+    <link name="${namespace}oak_left_camera_optical_frame"/>
+    <joint name="${namespace}oak_left_camera_optical_joint" type="fixed">
       <origin xyz="0 0 0" rpy="-${pi/2} 0.0 -${pi/2}"/>
-      <parent link="oak_left_camera_frame"/>
-      <child link="oak_left_camera_optical_frame"/>
+      <parent link="${namespace}oak_left_camera_frame"/>
+      <child link="${namespace}oak_left_camera_optical_frame"/>
     </joint>
     <!-- right Camera -->
-    <link name="oak_right_camera_frame" />
-    <joint name="oak_right_camera_joint" type="fixed">
-      <parent link="${base_frame}"/>
-      <child link="oak_right_camera_frame"/>
+    <link name="${namespace}oak_right_camera_frame" />
+    <joint name="${namespace}oak_right_camera_joint" type="fixed">
+      <parent link="${namespace}${base_frame}"/>
+      <child link="${namespace}oak_right_camera_frame"/>
       <origin xyz="0 -${baseline/2} 0" rpy="0 0 0" />
     </joint>
-    <link name="oak_right_camera_optical_frame"/>
-    <joint name="oak_right_camera_optical_joint" type="fixed">
+    <link name="${namespace}oak_right_camera_optical_frame"/>
+    <joint name="${namespace}oak_right_camera_optical_joint" type="fixed">
       <origin xyz="0 0 0" rpy="-${pi/2} 0.0 -${pi/2}"/>
-      <parent link="oak_right_camera_frame"/>
-      <child link="oak_right_camera_optical_frame"/>
+      <parent link="${namespace}oak_right_camera_frame"/>
+      <child link="${namespace}oak_right_camera_optical_frame"/>
     </joint>
   </xacro:macro>

File: raph_description/urdf/raph_macros.xacro (robot description, xacro)
@@ -9,8 +9,8 @@
                        imu_translation:='-0.128 0 -0.0393'">
     <!--TODO specify accurate imu translation-->
-    <xacro:oak_camera parent="${link_prefix}base_link" base_frame="${link_prefix}oak_base_frame">
+    <xacro:oak_camera parent="${link_prefix}base_link" base_frame="oak_base_frame" namespace="${link_prefix}">
       <origin xyz="-0.05642 0.0 -0.076218" rpy="0 0 0" />
     </xacro:oak_camera>
-    <xacro:rplidar_s3 parent="${link_prefix}base_link">
+    <xacro:rplidar_s3 parent="${link_prefix}base_link" namespace="${link_prefix}">
       <origin xyz="-0.062106 0.0 0.011588" />
     </xacro:rplidar_s3>
@@ -357,5 +357,5 @@
         </lidar>
         <topic>${link_prefix}scan_raw</topic>
-        <gz_frame_id>laser_frame</gz_frame_id>
+        <gz_frame_id>${link_prefix}laser_frame</gz_frame_id>
       </sensor>
     </gazebo>
@@ -515,4 +515,17 @@
       </plugin>
     </gazebo>
+    <!--Odometry publisher-->
+    <gazebo>
+      <plugin
+        filename="gz-sim-odometry-publisher-system"
+        name="gz::sim::systems::OdometryPublisher">
+        <odom_frame>${link_prefix}odom</odom_frame>
+        <robot_base_frame>${link_prefix}base_footprint</robot_base_frame>
+        <odom_publish_frequency>50</odom_publish_frequency>
+        <odom_topic>${link_prefix}odom</odom_topic>
+        <tf_topic>/tf</tf_topic>
+        <gaussian_noise>0.001</gaussian_noise>
+      </plugin>
+    </gazebo>
   </xacro:macro>
   <xacro:macro name="raph_sim"
