Commit message: feat: Add oak_stereo_camera_optical_frame to URDF

File: raph_description/urdf/include/oak_macro.xacro (robot description, xacro)
@@ -44,4 +44,10 @@
       <child link="${namespace}oak_left_camera_optical_frame"/>
     </joint>
+    <link name="${namespace}oak_stereo_camera_optical_frame" />
+    <joint name="${namespace}oak_stereo_camera_optical_joint" type="fixed">
+      <origin xyz="0 0 0" rpy="${pi/2} 0.0 ${pi/2}"/>
+      <parent link="${namespace}oak_left_camera_frame"/>
+      <child link="${namespace}oak_stereo_camera_optical_frame"/>
+    </joint>
     <!-- right Camera -->
     <link name="${namespace}oak_right_camera_frame" />

Commit message: fix: IMU frame orientation for upside-down camera setup

File: raph_description/urdf/include/oak_macro.xacro (robot description, xacro)
@@ -16,5 +16,5 @@
       <parent link="${namespace}${base_frame}"/>
       <child link="${namespace}oak_imu_frame"/>
-      <origin xyz="0.0 -0.015 -0.013662" rpy="0.0 ${pi/2} 0.0" />
+      <origin xyz="0.0 -0.015 -0.013662" rpy="0.0 -${pi/2} 0.0" />
     </joint>
     <!-- RGB Camera -->
