Commit message: Add all necessary gazebo configuration to urdf

File: raph_description/urdf/raph_macros.xacro (robot description, xacro)
@@ -17,4 +17,12 @@
     <xacro:macro name="servo_link" params="name">
       <link name="${link_prefix}servo_${name}_link">
+        <inertial>
+          <mass value="0.055"/>
+          <origin xyz="0 0 0"/>
+          <inertia
+            ixx="0.000001" ixy="0.0" ixz="0.0"
+            iyy="0.000001" iyz="0.0"
+            izz="0.000001"/>
+        </inertial>
         <visual>
           <origin xyz="0 0 0" rpy="0 0 ${pi/2}"/>
@@ -33,4 +41,12 @@
     <xacro:macro name="wheel_link" params="name">
       <link name="${link_prefix}wheel_${name}_link">
+        <inertial>
+          <mass value="0.5"/>
+          <origin xyz="0 0 0"/>
+          <inertia
+            ixx="0.002079" ixy="0.0" ixz="0.0"
+            iyy="0.002079" iyz="0.0"
+            izz="0.004158"/>
+        </inertial>
         <visual>
           <origin xyz="0 0 0" rpy="0 0 ${pi/2}"/>
@@ -52,4 +68,12 @@
     </xacro:if>
     <link name="${link_prefix}base_link">
+      <inertial>
+        <mass value="3.0"/>
+        <origin xyz="-0.019662 0.011643 -0.031802"/>
+        <inertia
+          ixx="0.02" ixy="0.001177" ixz="-0.0008871"
+          iyy="0.02" iyz="0.0002226"
+          izz="0.03"/>
+      </inertial>
       <visual>
         <origin xyz="-0.074211 0 -0.031076" rpy="0 0 ${pi/2}"/>
@@ -138,3 +162,323 @@
     </joint>
   </xacro:macro>
+  <!-- RAPH GAZEBO -->
+  <xacro:macro name="raph_gazebo"
+               params="robot_ns:=''">
+    <xacro:property name="link_prefix" value=""/>
+    <xacro:property name="joint_prefix" value=""/>
+    <xacro:if value="${robot_ns != '' and robot_ns != '/'}">
+      <xacro:property name="link_prefix" value="${robot_ns}/"/>
+      <xacro:property name="joint_prefix" value="${robot_ns}/"/>
+    </xacro:if>
+    <!-- base ODE properties -->
+    <gazebo reference="${link_prefix}base_footprint">
+      <collision>
+        <surface>
+          <friction>
+            <ode>
+              <mu>0.3</mu>
+              <mu2>0.3</mu2>
+            </ode>
+            <bullet>
+              <friction>0.3</friction>
+              <friction2>0.3</friction2>
+              <rolling_friction>0.1</rolling_friction>
+            </bullet>
+          </friction>
+        </surface>
+      </collision>
+    </gazebo>
+    <gazebo reference="${link_prefix}base_link">
+      <collision>
+        <surface>
+          <friction>
+            <ode>
+              <mu>0.3</mu>
+              <mu2>0.3</mu2>
+            </ode>
+            <bullet>
+              <friction>0.3</friction>
+              <friction2>0.3</friction2>
+              <rolling_friction>0.1</rolling_friction>
+            </bullet>
+          </friction>
+        </surface>
+      </collision>
+    </gazebo>
+    <!-- servo ODE properties -->
+    <gazebo reference="${link_prefix}servo_l_link">
+      <collision>
+        <surface>
+          <friction>
+            <ode>
+              <mu>0.3</mu>
+              <mu2>0.3</mu2>
+            </ode>
+            <bullet>
+              <friction>0.3</friction>
+              <friction2>0.3</friction2>
+              <rolling_friction>0.1</rolling_friction>
+            </bullet>
+          </friction>
+        </surface>
+      </collision>
+    </gazebo>
+    <gazebo reference="${link_prefix}servo_r_link">
+      <collision>
+        <surface>
+          <friction>
+            <ode>
+              <mu>0.3</mu>
+              <mu2>0.3</mu2>
+            </ode>
+            <bullet>
+              <friction>0.3</friction>
+              <friction2>0.3</friction2>
+              <rolling_friction>0.1</rolling_friction>
+            </bullet>
+          </friction>
+        </surface>
+      </collision>
+    </gazebo>
+    <!-- wheel ODE properties -->
+    <gazebo reference="${link_prefix}wheel_fl_link">
+      <collision>
+        <surface>
+          <friction>
+            <ode>
+              <mu>1</mu>
+              <mu2>1</mu2>
+              <slip1>0.035</slip1>
+              <slip2>0</slip2>
+              <fdir1>0 0 1</fdir1>
+            </ode>
+            <bullet>
+              <friction>1</friction>
+              <friction2>1</friction2>
+              <rolling_friction>0.1</rolling_friction>
+            </bullet>
+          </friction>
+        </surface>
+      </collision>
+    </gazebo>
+    <gazebo reference="${link_prefix}wheel_fr_link">
+      <collision>
+        <surface>
+          <friction>
+            <ode>
+              <mu>1</mu>
+              <mu2>1</mu2>
+              <slip1>0.035</slip1>
+              <slip2>0</slip2>
+              <fdir1>0 0 1</fdir1>
+            </ode>
+            <bullet>
+              <friction>1</friction>
+              <friction2>1</friction2>
+              <rolling_friction>0.1</rolling_friction>
+            </bullet>
+          </friction>
+        </surface>
+      </collision>
+    </gazebo>
+    <gazebo reference="${link_prefix}wheel_rl_link">
+      <collision>
+        <surface>
+          <friction>
+            <ode>
+              <mu>1</mu>
+              <mu2>1</mu2>
+              <slip1>0.035</slip1>
+              <slip2>0</slip2>
+              <fdir1>0 0 1</fdir1>
+            </ode>
+            <bullet>
+              <friction>1</friction>
+              <friction2>1</friction2>
+              <rolling_friction>0.1</rolling_friction>
+            </bullet>
+          </friction>
+        </surface>
+      </collision>
+    </gazebo>
+    <gazebo reference="${link_prefix}wheel_rr_link">
+      <collision>
+        <surface>
+          <friction>
+            <ode>
+              <mu>1</mu>
+              <mu2>1</mu2>
+              <slip1>0.035</slip1>
+              <slip2>0</slip2>
+              <fdir1>0 0 1</fdir1>
+            </ode>
+            <bullet>
+              <friction>1</friction>
+              <friction2>1</friction2>
+              <rolling_friction>0.1</rolling_friction>
+            </bullet>
+          </friction>
+        </surface>
+      </collision>
+    </gazebo>
+    <!-- Joint state publisher -->
+    <gazebo>
+      <plugin
+        filename="libgz-sim-joint-state-publisher-system.so"
+        name="gz::sim::systems::JointStatePublisher">
+        <topic>${link_prefix}joint_states</topic>
+      </plugin>
+    </gazebo>
+    <!-- TODO adjust sensor configurations -->
+    <!-- RPLidar S3 sensor -->
+    <gazebo reference="laser_frame">
+      <sensor name="rplidar_s3" type="gpu_lidar">
+        <visualize>true</visualize>
+        <update_rate>15</update_rate>
+        <lidar>
+          <scan>
+            <horizontal>
+              <samples>720</samples>
+              <resolution>1</resolution>
+              <min_angle>-3.14159</min_angle>
+              <max_angle>3.14159</max_angle>
+            </horizontal>
+          </scan>
+          <range>
+            <min>0.10</min>
+            <max>25.0</max>
+            <resolution>0.01</resolution>
+          </range>
+          <noise>
+            <type>gaussian</type>
+            <mean>0.0</mean>
+            <stddev>0.01</stddev>
+          </noise>
+        </lidar>
+        <topic>${link_prefix}scan</topic>
+        <gz_frame_id>laser_frame</gz_frame_id>
+      </sensor>
+    </gazebo>
+    <!-- OAK-D Pro W RGB camera -->
+    <gazebo reference="${link_prefix}oak_rgb_camera_frame">
+      <sensor name="oak_rgb_camera" type="camera">
+        <camera name="oak_rgb">
+          <horizontal_fov>1.204</horizontal_fov>
+          <image>
+            <width>1920</width>
+            <height>1080</height>
+            <format>R8G8B8</format>
+          </image>
+          <clip>
+            <near>0.1</near>
+            <far>100</far>
+          </clip>
+          <noise>
+            <type>gaussian</type>
+            <mean>0.0</mean>
+            <stddev>0.007</stddev>
+          </noise>
+        </camera>
+        <always_on>1</always_on>
+        <update_rate>30</update_rate>
+        <visualize>true</visualize>
+        <topic>${link_prefix}oak/rgb/image_raw</topic>
+        <gz_frame_id>${link_prefix}oak_rgb_camera_optical_frame</gz_frame_id>
+      </sensor>
+    </gazebo>
+    <!-- OAK-D Pro W Depth camera -->
+    <gazebo reference="${link_prefix}oak_rgb_camera_frame">
+      <sensor name="oak_depth_camera" type="depth_camera">
+        <camera name="oak_depth">
+          <horizontal_fov>1.204</horizontal_fov>
+          <image>
+            <width>1280</width>
+            <height>720</height>
+            <format>R_FLOAT32</format>
+          </image>
+          <clip>
+            <near>0.1</near>
+            <far>10.0</far>
+          </clip>
+          <noise>
+            <type>gaussian</type>
+            <mean>0.0</mean>
+            <stddev>0.01</stddev>
+          </noise>
+        </camera>
+        <always_on>1</always_on>
+        <update_rate>15</update_rate>
+        <visualize>true</visualize>
+        <topic>${link_prefix}oak/depth/image_raw</topic>
+        <gz_frame_id>${link_prefix}oak_right_camera_frame</gz_frame_id>
+      </sensor>
+    </gazebo>
+    <!-- IMU sensor -->
+    <gazebo reference="${link_prefix}imu_frame">
+      <sensor type="imu" name="raph_imu_sensor">
+        <update_rate>100</update_rate>
+        <visualize>true</visualize>
+        <topic>${link_prefix}imu/data</topic>
+        <always_on>1</always_on>
+        <gz_frame_id>${link_prefix}imu_frame</gz_frame_id>
+      </sensor>
+    </gazebo>
+    <!-- All-wheel drive with rear steering plugin -->
+    <gazebo>
+      <plugin
+        filename="gz-sim-ackermann-steering-system"
+        name="gz::sim::systems::AckermannSteering">
+        <left_steering_joint>${joint_prefix}servo_l_joint</left_steering_joint>
+        <right_steering_joint>${joint_prefix}servo_r_joint</right_steering_joint>
+        <left_joint>${joint_prefix}wheel_rl_joint</left_joint>
+        <right_joint>${joint_prefix}wheel_rr_joint</right_joint>
+        <left_joint>${joint_prefix}wheel_fl_joint</left_joint>
+        <right_joint>${joint_prefix}wheel_fr_joint</right_joint>
+        <!-- TODO make sure that the params are set correctly -->
+        <wheelbase>0.379</wheelbase>
+        <wheel_separation>0.38</wheel_separation>
+        <wheel_radius>0.091</wheel_radius>
+        <steering_limit>1.48353</steering_limit>
+        <!-- <kingpin_width>change_this</kingpin_width> -->
+        <min_steering_angle>-1.5708</min_steering_angle>
+        <max_steering_angle>1.5708</max_steering_angle>
+        <topic>${link_prefix}cmd_vel</topic>
+        <odom_topic>${link_prefix}odom</odom_topic>
+        <tf_topic>${link_prefix}tf</tf_topic>
+        <frame_id>odom</frame_id>
+        <child_frame_id>${link_prefix}base_footprint</child_frame_id>
+        <odom_publish_frequency>50</odom_publish_frequency>
+      </plugin>
+    </gazebo>
+    <gazebo>
+      <plugin
+        filename="libraph_gz_ackermann_plugin.so"
+        name="raph_gz_plugins::AckermannToTwist">
+        <robotNamespace>${link_prefix}</robotNamespace>
+        <!-- TODO make sure that the params are set correctly -->
+        <wheelbase>0.379</wheelbase>
+        <maxSteeringAngle>1.5708</maxSteeringAngle>
+      </plugin>
+    </gazebo>
+  </xacro:macro>
+  <xacro:macro name="raph_sim"
+               params="fixed:=false
+                       robot_ns:=''">
+    <xacro:property name="link_prefix" value=""/>
+    <xacro:property name="joint_prefix" value=""/>
+    <xacro:if value="${robot_ns != '' and robot_ns != '/'}">
+      <xacro:property name="link_prefix" value="${robot_ns}/"/>
+      <xacro:property name="joint_prefix" value="${robot_ns}/"/>
+    </xacro:if>
+    <xacro:raph link_prefix="${link_prefix}" joint_prefix="${joint_prefix}"/>
+    <xacro:raph_gazebo robot_ns="${robot_ns}"/>
+    <xacro:if value="${fixed}">
+      <link name="world"/>
+      <joint name="fixed" type="fixed">
+        <parent link="world"/>
+        <child link="${link_prefix}base_footprint"/>
+        <origin xyz="0.0 0.0 1.0"/>
+      </joint>
+    </xacro:if>
+  </xacro:macro>
 </robot>

Commit message: Adjust friction and servo speed

File: raph_description/urdf/raph_macros.xacro (robot description, xacro)
@@ -125,5 +125,5 @@
       <axis xyz="0 1 0"/>
       <limit effort="2.0" velocity="6.0"/>
-      <dynamics friction="0.3125" damping="0.1"/>
+      <dynamics friction="0.5" damping="0.2"/>
     </joint>
     <joint name="${joint_prefix}wheel_rl_joint" type="continuous">
@@ -133,5 +133,5 @@
       <axis xyz="0 1 0"/>
       <limit effort="2.0" velocity="6.0"/>
-      <dynamics friction="0.3125" damping="0.1"/>
+      <dynamics friction="0.5" damping="0.2"/>
     </joint>
     <joint name="${joint_prefix}wheel_fr_joint" type="continuous">
@@ -141,5 +141,5 @@
       <axis xyz="0 -1 0"/>
       <limit effort="2.0" velocity="6.0"/>
-      <dynamics friction="0.3125" damping="0.1"/>
+      <dynamics friction="0.5" damping="0.2"/>
     </joint>
     <joint name="${joint_prefix}wheel_rr_joint" type="continuous">
@@ -149,5 +149,5 @@
       <axis xyz="0 -1 0"/>
       <limit effort="2.0" velocity="6.0"/>
-      <dynamics friction="0.3125" damping="0.1"/>
+      <dynamics friction="0.5" damping="0.2"/>
     </joint>
     <joint name="${joint_prefix}imu_joint" type="fixed">
@@ -247,14 +247,13 @@
           <friction>
             <ode>
-              <mu>1</mu>
-              <mu2>1</mu2>
-              <slip1>0.035</slip1>
-              <slip2>0</slip2>
-              <fdir1>0 0 1</fdir1>
-            </ode>
-            <bullet>
-              <friction>1</friction>
-              <friction2>1</friction2>
-              <rolling_friction>0.1</rolling_friction>
+              <mu>2.0</mu>
+              <mu2>2.0</mu2>
+              <slip1>0.01</slip1>
+              <slip2>0.01</slip2>
+            </ode>
+            <bullet>
+              <friction>2.0</friction>
+              <friction2>2.0</friction2>
+              <rolling_friction>0.2</rolling_friction>
             </bullet>
           </friction>
@@ -267,14 +266,13 @@
           <friction>
             <ode>
-              <mu>1</mu>
-              <mu2>1</mu2>
-              <slip1>0.035</slip1>
-              <slip2>0</slip2>
-              <fdir1>0 0 1</fdir1>
-            </ode>
-            <bullet>
-              <friction>1</friction>
-              <friction2>1</friction2>
-              <rolling_friction>0.1</rolling_friction>
+              <mu>2.0</mu>
+              <mu2>2.0</mu2>
+              <slip1>0.01</slip1>
+              <slip2>0.01</slip2>
+            </ode>
+            <bullet>
+              <friction>2.0</friction>
+              <friction2>2.0</friction2>
+              <rolling_friction>0.2</rolling_friction>
             </bullet>
           </friction>
@@ -287,14 +285,13 @@
           <friction>
             <ode>
-              <mu>1</mu>
-              <mu2>1</mu2>
-              <slip1>0.035</slip1>
-              <slip2>0</slip2>
-              <fdir1>0 0 1</fdir1>
-            </ode>
-            <bullet>
-              <friction>1</friction>
-              <friction2>1</friction2>
-              <rolling_friction>0.1</rolling_friction>
+              <mu>2.0</mu>
+              <mu2>2.0</mu2>
+              <slip1>0.01</slip1>
+              <slip2>0.01</slip2>
+            </ode>
+            <bullet>
+              <friction>2.0</friction>
+              <friction2>2.0</friction2>
+              <rolling_friction>0.2</rolling_friction>
             </bullet>
           </friction>
@@ -307,14 +304,13 @@
           <friction>
             <ode>
-              <mu>1</mu>
-              <mu2>1</mu2>
-              <slip1>0.035</slip1>
-              <slip2>0</slip2>
-              <fdir1>0 0 1</fdir1>
-            </ode>
-            <bullet>
-              <friction>1</friction>
-              <friction2>1</friction2>
-              <rolling_friction>0.1</rolling_friction>
+              <mu>2.0</mu>
+              <mu2>2.0</mu2>
+              <slip1>0.01</slip1>
+              <slip2>0.01</slip2>
+            </ode>
+            <bullet>
+              <friction>2.0</friction>
+              <friction2>2.0</friction2>
+              <rolling_friction>0.2</rolling_friction>
             </bullet>
           </friction>
@@ -454,6 +450,6 @@
         <topic>/${joint_prefix}servo_l_joint/cmd_pos</topic>
         <use_velocity_commands>true</use_velocity_commands>
-        <cmd_max>1</cmd_max>
-        <cmd_min>-1</cmd_min>
+        <cmd_max>3.0</cmd_max>
+        <cmd_min>-3.0</cmd_min>
       </plugin>
     </gazebo>
@@ -463,6 +459,6 @@
         <topic>/${joint_prefix}servo_r_joint/cmd_pos</topic>
         <use_velocity_commands>true</use_velocity_commands>
-        <cmd_max>1</cmd_max>
-        <cmd_min>-1</cmd_min>
+        <cmd_max>3.0</cmd_max>
+        <cmd_min>-3.0</cmd_min>
       </plugin>
     </gazebo>
